Commit message: Changed Arm DOF3 to DOF4

File: urdf/humanoid.xacro (robot description, xacro)
@@ -158,14 +158,15 @@
     </inertial>
   </link>
-  <joint name="left_hand_joint" type="fixed">
+  <joint name="left_hand_joint" type="revolute">
     <parent link="left_forearm"/>
     <child link="left_hand"/>
-    <origin xyz="0 0 0.1" rpy="0 0  0"/>
-    <axis xyz="0 0 0"/>
+    <origin xyz="0 0 0.2" rpy="0 0  0"/>
+  	<limit effort="300" velocity="3" lower="-3.14" upper="3.14"/>
+    <axis xyz="0 0 1"/>
     <dynamics damping="0.7"/>
   </joint>
 `  <link name="left_hand">
      <collision>
-      <origin xyz="0 0 0.1" rpy="0 0 0"/>
+      <origin xyz="0 0 0" rpy="0 0 0"/>
       <geometry>
     	  <sphere radius="0.03" />
@@ -173,5 +174,5 @@
     </collision>
     <visual>
-      <origin xyz="0 0 0.1" rpy="0 0 0"/>
+      <origin xyz="0 0 0" rpy="0 0 0"/>
       <geometry>
           <sphere radius="0.03" />
@@ -180,5 +181,5 @@
     </visual>
     <inertial>
-      <origin xyz="0 0 0.1" rpy="0 0 0"/>
+      <origin xyz="0 0 0" rpy="0 0 0"/>
       <mass value="${mass}"/>
       <inertia
@@ -276,14 +277,15 @@
     </inertial>
   </link>
-  <joint name="right_hand_joint" type="fixed">
+  <joint name="right_hand_joint" type="revolute">
     <parent link="right_forearm"/>
     <child link="right_hand"/>
-    <origin xyz="0 0 0.1" rpy="0 0  0"/>
-    <axis xyz="0 0 0"/>
-    <dynamics damping="0.7"/>
-  </joint>
-`  <link name="right_hand">
-     <collision>
-      <origin xyz="0 0 0.1" rpy="0 0 0"/>
+    <origin xyz="0 0 0.2" rpy="0 0  0"/>
+  	<limit effort="300" velocity="3" lower="-3.14" upper="3.14"/>
+    <axis xyz="0 0 1"/>
+    <dynamics damping="0.7"/>
+  </joint>
+  <link name="right_hand">
+     <collision>
+      <origin xyz="0 0 0" rpy="0 0 0"/>
       <geometry>
     	  <sphere radius="0.03" />
@@ -291,5 +293,5 @@
     </collision>
     <visual>
-      <origin xyz="0 0 0.1" rpy="0 0 0"/>
+      <origin xyz="0 0 0" rpy="0 0 0"/>
       <geometry>
           <sphere radius="0.03" />
@@ -298,5 +300,5 @@
     </visual>
     <inertial>
-      <origin xyz="0 0 0.1" rpy="0 0 0"/>
+      <origin xyz="0 0 0" rpy="0 0 0"/>
       <mass value="${mass}"/>
       <inertia
